File: schematic/schematic/main.sch (EAGLE design)
At the start: 36 parts, among them IC1 STM32F103C8T6, IC2 ESP8266, IC3 DRV8836, IC4 MCP73831, IC5 MCP1825S-3302E/DB, Y1 8MHz

Commit message: Correct errors
Parts:
- removed IC2: ESP8266, esp8266modules:ESP8266
- removed JP1, JP2: (no value), pinhead:PINHD-1X4/90
- removed PWR_LED: (no value), eagle-ltspice:LED_ESML0603
- added BLU: BLUE, SparkFun-LED:LED-BLUE0603
- added C10, C11, C13, C14, C15: 100nF, SparkFun-Capacitors:CAP0603-CAP
- added C16: 4.7uF, SparkFun-Capacitors:CAP0603-CAP
- added C17: 10nF, SparkFun-Capacitors:CAP0603-CAP
- added C18: 500nF, SparkFun-Capacitors:CAP0603-CAP
- added J3: (no value), SparkFun-Connectors:CONN_05X2PTH
- added PWR: (no value), eagle-ltspice:LED_ESML0603
- added R10, R11, R12, R9: 10K, rcl:R-EU_R0603
- added R13, R14, R15: 330, resistor:R-EU_R0603
- added TP1: TP5P5-25-13, testpad:TP5P5-25-13
- added U1: (no value), esp8266modules:ESP12
- added WHT: WHITE, SparkFun-LED:LED-WHITE0603
- IC5: value MCP1825S-3302E/DB -> MCP1826S-3302E/DB; device MCP1825S-3302E_DB:MCP1825S-3302E/DB -> MCP1826S-3302E_DB:MCP1826S-3302E/DB
- renumbered CHG_LED to CHG
Connections:
- net LEDB renamed PB15(LEDB)
- net LEDG renamed PB14(LEDG)
- net LEDR renamed PB13(LEDR)
- net PHA1 renamed PB0(PHA1)
- net PHA2 renamed PB1(PHA2)
- net PWM1 renamed PB8(PWM1)
- net PWM2 renamed PB9(PWM2)
- removed net D+: IC1.PA12
- removed net D-: IC1.PA11
- removed net N$11: C8.2, C9.2
- removed net N$12: JP1.2
- removed net N$13: JP1.3
- removed net N$17: JP1.4
- removed net PA11: R7.1
- removed net PA12: R5.2, R6.1
- new net 3V3: R12.1, U1.VCC
- new net CH_PD: R12.2, U1.CH_PD
- new net GPIO15: R10.2, U1.GPIO15
- new net GPIO5: R9.2, U1.GPIO5
- new net MODE(PC14): IC1.PC14-OSC32_IN
- new net N$18: R13.1, WHT.A
- new net N$19: BLU.A, R14.1
- new net PA0(T2C1): IC1.PA0, J3.2
- new net PA1(T2C2): IC1.PA1, J3.4
- new net PA10(RX): IC1.PA10, U1.TX
- new net PA11(D-): IC1.PA11, R7.1
- new net PA12(D+): IC1.PA12, R5.2, R6.1
- new net PA13(SWDIO): IC1.PA13, TP1C.TP
- new net PA14(SW_CLK): IC1.PA14, TP1D.TP
- new net PA2(TX): IC1.PA2, J3.6
- new net PA3(RX): IC1.PA3, J3.8
- new net PA4(BLU): IC1.PA4, R14.2
- new net PA5(WHT): IC1.PA5, R13.2
- new net PA9(TX): IC1.PA9, U1.RX
- new net PB10(SCL): IC1.PB10, J3.7
- new net PB11(SDA): IC1.PB11, J3.9
- new net PB6(SCL): IC1.PB6, J3.3
- new net PB7(SDA): IC1.PB7, J3.5
- new net VDD1: IC1.VDD1, J3.1
- new net VDDA: C17.2, C18.2, IC1.VDDA
- new net VSS1: IC1.VSS1, J3.10
- new net VSSA: C17.1, C18.1, IC1.VSSA
- net +3V3: now also C10.2, C11.2, C13.2, C14.2, C15.2, C16.1, IC1.VDD2, IC1.VDD3, TP1B.TP; no longer H2.MOUNT, IC2.VCC
- net BOOT0: now also R9.1
- net BOOT1: now also R11.2
- net GND: now also BLU.C, C10.1, C11.1, C13.1, C14.1, C15.1, C16.2, C8.2, C9.2, H2.MOUNT, IC1.VSS2, IC1.VSS3, IC5.GND_(TAB), PWR.C, R10.1, R11.1, TP1E.TP, U1.GND, WHT.C; no longer IC2.GND, PWR_LED.C, USB.ID
- net MODE: no longer IC1.PC14-OSC32_IN
- net N$1: now also C12.2, R15.2; no longer JP1.1
- net N$10: now also PWR.A; no longer PWR_LED.A
- net N$15: now also R15.1; no longer C12.2
- net RESET: now also U1.GPIO4
- net VBATT: now also TP1A.TP
Other:
- note added: "Battery Mount"
- note added: "Battery Switch"
- note added: "ESP8266"
- note added: "Expansion Slot"
- note added: "Micro USB"
- note added: "Microcontroller"
- note added: "Oscillator Circuit"
- note added: "Power Supply"
- note added: "RGB LED"
- note added: "Reset Switch"
- note added: "SWD"
- moved on the sheet: C1, C12, C4, C5, C6, C7, C8, C9, D1, H2, H3, IC3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
