File: schematic/schematic/HiveX-Schematic-09.sch (EAGLE design)
At the start: 53 parts, among them IC1 STM32F103C8T6, IC3 DRV8836, IC4 MCP73831, IC5 MCP1826S-3302E/DB, Y1 8MHz

Commit message: Updated schematic
Parts:
- removed C16: 4.7uF, SparkFun-Capacitors:CAP0603-CAP
- removed C17: 10nF, SparkFun-Capacitors:CAP0603-CAP
- removed C18: 500nF, SparkFun-Capacitors:CAP0603-CAP
- removed J3: (no value), SparkFun-Connectors:CONN_05X2PTH
- removed R15: 330, resistor:R-EU_R0603
- removed S1: (no value), eswitch-tact:TL3302-J
- removed TP1: TP5P5-25-13, testpad:TP5P5-25-13
- added M1, M2: (no value), SparkFun-Connectors:JST_2MM_MALE
- added RST: (no value), eswitch-tact:TL3302-J
- BLU: value BLUE -> Blue
- C14: value 100nF -> 10uF
- CHG: value (none) -> Red
- J1: device SparkFun-Connectors:JST_2MM_MALE -> SparkFun-Connectors:CONN_05X2PTH
- J2: value (none) -> TP5P5-25-13; device SparkFun-Connectors:JST_2MM_MALE -> testpad:TP5P5-25-13
- PWR: value (none) -> Yellow
- WHT: value WHITE -> White
- renumbered U1 to IC2
Connections:
- net VCC renamed 5V
- removed net +3V3: C10.2, C11.2, C13.2, C14.2, C15.2, C16.1, C6.1, C7.1, D1.A, IC1.VBAT, IC1.VDD2, IC1.VDD3, IC5.VOUT, R8.2
- removed net MODE(PC14): IC1.PC14-OSC32_IN
- removed net N$1: C12.2, R15.2
- removed net N$15: R15.1, S1.1
- removed net N$21: TP1B.TP
- removed net NRST: IC2.GPIO4
- removed net PC15: IC1.PC15-OSC32_OUT
- removed net VDD1: IC1.VDD1, J3.1
- removed net VDDA: C17.2, C18.2, IC1.VDDA
- removed net VSS1: IC1.VSS1, J3.10
- removed net VSSA: C17.1, C18.1, IC1.VSSA
- net 3V3: now also C10.2, C11.2, C13.2, C14.2, C15.2, C6.1, C7.1, D1.A, IC1.VBAT, IC1.VDD1, IC1.VDD2, IC1.VDD3, IC1.VDDA, IC5.VOUT, J1.1, J2B.TP, R8.2
- net GND: now also C12.2, IC1.VSS1, IC1.VSSA, J1.10, J2E.TP, RST.1; no longer C16.2, TP1E.TP
- net MODE: now also IC1.PC14-OSC32_IN
- net N$2: now also M1.+; no longer J1.+
- net N$3: now also M2.-; no longer J2.-
- net N$4: now also M1.-; no longer J1.-
- net N$5: now also M2.+; no longer J2.+
- net PA0(T2C1): now also J1.2; no longer J3.2
- net PA1(T2C2): now also J1.4; no longer J3.4
- net PA13(SWDIO): now also J2C.TP; no longer TP1C.TP
- net PA14(SW_CLK): now also J2D.TP; no longer TP1D.TP
- net PA2(TX): now also J1.6; no longer J3.6
- net PA3(RX): now also J1.8; no longer J3.8
- net PB10(SCL): now also J1.7; no longer J3.7
- net PB11(SDA): now also J1.9; no longer J3.9
- net PB6(SCL): now also J1.3; no longer J3.3
- net PB7(SDA): now also J1.5; no longer J3.5
- net RESET: now also IC2.GPIO4, RST.2; no longer S1.2
- net VBATT: now also J2A.TP; no longer TP1A.TP
Other:
- note removed: "Red"
- note removed: "Yellow"
- moved on the sheet: BLU, C1, C10, C11, C12, C13, C14, C15, D1, IC3, R13, R14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
